File: doc/pcb/term.sch (KiCad schematic (older format))
At the start: 18 parts, among them U1 LM35-LP, U2 LM1117-3.3, U3 STM32F030F4Px, U4 CA56-12CGKWA

Commit message: new pcb as credit card
Parts:
- removed BT1: Battery, Connector_PinHeader_2.54mm:PinHeader_1x02_P2.54mm_Vertical, symbol Device:Battery
- added J1: USB_B_Micro, Connector_USB:USB_Micro-B_Molex-105017-0001, symbol Connector:USB_B_Micro
- C1: footprint Capacitor_THT:C_Disc_D3.0mm_W1.6mm_P2.50mm -> Capacitor_THT:C_Disc_D10.5mm_W5.0mm_P5.00mm
- C2, C3: footprint Capacitor_THT:C_Disc_D3.0mm_W1.6mm_P2.50mm -> Capacitor_THT:C_Disc_D8.0mm_W5.0mm_P7.50mm
- L1, R1, R10, R2, R3, R4, R5, R6, R7, R9: footprint Resistor_THT:R_Axial_DIN0204_L3.6mm_D1.6mm_P2.54mm_Vertical -> Resistor_THT:R_Axial_DIN0207_L6.3mm_D2.5mm_P10.16mm_Horizontal
Connections:
- net GND: now also J1.5 (GND)
- net +9V renamed +5V
- net +5V: now also J1.1 (VBUS)
- no-connect marks 4 -> 8
Changed lines of the file:
@@
 F 0 "R2" H 5020 2746 50  0000 L CNN
 F 1 "10k" H 5020 2655 50  0000 L CNN
-F 2 "Resistor_THT:R_Axial_DIN0204_L3.6mm_D1.6mm_P2.54mm_Vertical" V 4880 2700 50  0001 C CNN
+F 2 "Resistor_THT:R_Axial_DIN0207_L6.3mm_D2.5mm_P10.16mm_Horizontal" V 4880 2700 50  0001 C CNN
 F 3 "~" H 4950 2700 50  0001 C CNN
 	1    4950 2700
@@
 F 0 "R1" H 4270 3696 50  0000 L CNN
 F 1 "10k" H 4270 3605 50  0000 L CNN
-F 2 "Resistor_THT:R_Axial_DIN0204_L3.6mm_D1.6mm_P2.54mm_Vertical" V 4130 3650 50  0001 C CNN
+F 2 "Resistor_THT:R_Axial_DIN0207_L6.3mm_D2.5mm_P10.16mm_Horizontal" V 4130 3650 50  0001 C CNN
 F 3 "~" H 4200 3650 50  0001 C CNN
 	1    4200 3650
@@
 D4
 $Comp
-L Device:Battery BT1
-U 1 1 5D351A65
-P 2400 2600
-F 0 "BT1" H 2508 2646 50  0000 L CNN
-F 1 "Battery" H 2508 2555 50  0000 L CNN
-F 2 "Connector_PinHeader_2.54mm:PinHeader_1x02_P2.54mm_Vertical" V 2400 2660 50  0001 C CNN
-F 3 "~" V 2400 2660 50  0001 C CNN
-	1    2400 2600
-	1    0    0    -1
-$EndComp
-$Comp
 L Regulator_Linear:LM1117-3.3 U2
 U 1 1 5D3528B6
@@
 F 0 "C1" H 2965 2546 50  0000 L CNN
 F 1 "100n" H 2965 2455 50  0000 L CNN
-F 2 "Capacitor_THT:C_Disc_D3.0mm_W1.6mm_P2.50mm" H 2888 2350 50  0001 C CNN
+F 2 "Capacitor_THT:C_Disc_D10.5mm_W5.0mm_P5.00mm" H 2888 2350 50  0001 C CNN
 F 3 "~" H 2850 2500 50  0001 C CNN
 	1    2850 2500
@@
 F 0 "C2" H 4165 2546 50  0000 L CNN
 F 1 "100n" H 4165 2455 50  0000 L CNN
-F 2 "Capacitor_THT:C_Disc_D3.0mm_W1.6mm_P2.50mm" H 4088 2350 50  0001 C CNN
+F 2 "Capacitor_THT:C_Disc_D8.0mm_W5.0mm_P7.50mm" H 4088 2350 50  0001 C CNN
 F 3 "~" H 4050 2500 50  0001 C CNN
 	1    4050 2500
@@
 	2850 2800 3450 2800
 $Comp
-L power:+9V #PWR0106
+L power:+5V #PWR0106
 U 1 1 5D35634A
 P 2400 2350
 F 0 "#PWR0106" H 2400 2200 50  0001 C CNN
-F 1 "+9V" H 2415 2523 50  0000 C CNN
+F 1 "+5V" H 2415 2523 50  0000 C CNN
 F 2 "" H 2400 2350 50  0001 C CNN
 F 3 "" H 2400 2350 50  0001 C CNN
@@
 F 0 "L1" H 5653 2696 50  0000 L CNN
 F 1 "10uH" H 5653 2605 50  0000 L CNN
-F 2 "Resistor_THT:R_Axial_DIN0204_L3.6mm_D1.6mm_P2.54mm_Vertical" H 5600 2650 50  0001 C CNN
+F 2 "Resistor_THT:R_Axial_DIN0207_L6.3mm_D2.5mm_P10.16mm_Horizontal" H 5600 2650 50  0001 C CNN
 F 3 "~" H 5600 2650 50  0001 C CNN
 	1    5600 2650
@@
 $EndComp
 $Comp
-L power:+9V #PWR01
+L power:+5V #PWR01
 U 1 1 5D463DDB
 P 7100 2350
 F 0 "#PWR01" H 7100 2200 50  0001 C CNN
-F 1 "+9V" H 7115 2523 50  0000 C CNN
+F 1 "+5V" H 7115 2523 50  0000 C CNN
 F 2 "" H 7100 2350 50  0001 C CNN
 F 3 "" H 7100 2350 50  0001 C CNN
@@
 F 0 "C3" V 6998 3250 50  0000 C CNN
 F 1 "100n" V 7089 3250 50  0000 C CNN
-F 2 "Capacitor_THT:C_Disc_D3.0mm_W1.6mm_P2.50mm" H 7288 3100 50  0001 C CNN
+F 2 "Capacitor_THT:C_Disc_D8.0mm_W5.0mm_P7.50mm" H 7288 3100 50  0001 C CNN
 F 3 "~" H 7250 3250 50  0001 C CNN
 	1    7250 3250
@@
 F 0 "R5" V 6600 4000 50  0000 C CNN
 F 1 "470" V 6700 4000 50  0000 C CNN
-F 2 "Resistor_THT:R_Axial_DIN0204_L3.6mm_D1.6mm_P2.54mm_Vertical" V 6080 3400 50  0001 C CNN
+F 2 "Resistor_THT:R_Axial_DIN0207_L6.3mm_D2.5mm_P10.16mm_Horizontal" V 6080 3400 50  0001 C CNN
 F 3 "~" H 6150 3400 50  0001 C CNN
 	1    6150 3400
@@
 F 0 "R6" V 6700 4100 50  0000 C CNN
 F 1 "470" V 6800 4100 50  0000 C CNN
-F 2 "Resistor_THT:R_Axial_DIN0204_L3.6mm_D1.6mm_P2.54mm_Vertical" V 6080 3500 50  0001 C CNN
+F 2 "Resistor_THT:R_Axial_DIN0207_L6.3mm_D2.5mm_P10.16mm_Horizontal" V 6080 3500 50  0001 C CNN
 F 3 "~" H 6150 3500 50  0001 C CNN
 	1    6150 3500
@@
 F 0 "R7" V 6800 4200 50  0000 C CNN
 F 1 "470" V 6900 4200 50  0000 C CNN
-F 2 "Resistor_THT:R_Axial_DIN0204_L3.6mm_D1.6mm_P2.54mm_Vertical" V 6080 3600 50  0001 C CNN
+F 2 "Resistor_THT:R_Axial_DIN0207_L6.3mm_D2.5mm_P10.16mm_Horizontal" V 6080 3600 50  0001 C CNN
 F 3 "~" H 6150 3600 50  0001 C CNN
 	1    6150 3600
@@
 F 0 "R9" V 6200 4650 50  0000 C CNN
 F 1 "470" V 6300 4650 50  0000 C CNN
-F 2 "Resistor_THT:R_Axial_DIN0204_L3.6mm_D1.6mm_P2.54mm_Vertical" V 6080 3800 50  0001 C CNN
+F 2 "Resistor_THT:R_Axial_DIN0207_L6.3mm_D2.5mm_P10.16mm_Horizontal" V 6080 3800 50  0001 C CNN
 F 3 "~" H 6150 3800 50  0001 C CNN
 	1    6150 3800
@@
 F 0 "R10" V 6300 4750 50  0000 C CNN
 F 1 "470" V 6400 4750 50  0000 C CNN
-F 2 "Resistor_THT:R_Axial_DIN0204_L3.6mm_D1.6mm_P2.54mm_Vertical" V 6080 3900 50  0001 C CNN
+F 2 "Resistor_THT:R_Axial_DIN0207_L6.3mm_D2.5mm_P10.16mm_Horizontal" V 6080 3900 50  0001 C CNN
 F 3 "~" H 6150 3900 50  0001 C CNN
 	1    6150 3900
@@
 F 0 "R3" V 4650 3800 50  0000 C CNN
 F 1 "470" V 4750 3800 50  0000 C CNN
-F 2 "Resistor_THT:R_Axial_DIN0204_L3.6mm_D1.6mm_P2.54mm_Vertical" V 4780 3800 50  0001 C CNN
+F 2 "Resistor_THT:R_Axial_DIN0207_L6.3mm_D2.5mm_P10.16mm_Horizontal" V 4780 3800 50  0001 C CNN
 F 3 "~" H 4850 3800 50  0001 C CNN
 	1    4850 3800
@@
 F 0 "R4" V 4950 3900 50  0000 C CNN
 F 1 "470" V 5050 3900 50  0000 C CNN
-F 2 "Resistor_THT:R_Axial_DIN0204_L3.6mm_D1.6mm_P2.54mm_Vertical" V 4780 3900 50  0001 C CNN
+F 2 "Resistor_THT:R_Axial_DIN0207_L6.3mm_D2.5mm_P10.16mm_Horizontal" V 4780 3900 50  0001 C CNN
 F 3 "~" H 4850 3900 50  0001 C CNN
 	1    4850 3900
@@
 Wire Wire Line
 	6000 3700 7500 3700
+$Comp
+L Connector:USB_B_Micro J1
+U 1 1 5D4BA4CA
+P 1800 2600
+F 0 "J1" H 1857 3067 50  0000 C CNN
+F 1 "USB_B_Micro" H 1857 2976 50  0000 C CNN
+F 2 "Connector_USB:USB_Micro-B_Molex-105017-0001" H 1950 2550 50  0001 C CNN
+F 3 "~" H 1950 2550 50  0001 C CNN
+	1    1800 2600
+	1    0    0    -1
+$EndComp
+Wire Wire Line
+	2100 2400 2400 2400
+Wire Wire Line
+	1800 3000 2400 3000
+Wire Wire Line
+	2400 3000 2400 2800
+NoConn ~ 1700 3000
+NoConn ~ 2100 2800
+NoConn ~ 2100 2700
+NoConn ~ 2100 2600
 $EndSCHEMATC

Commit message: little pcb corrections
Parts:
- J1: footprint Connector_USB:USB_Micro-B_Molex-105017-0001 -> Connector_USB:USB_Micro-B_Molex_47346-0001
Changed lines of the file:
@@
 F 0 "J1" H 1857 3067 50  0000 C CNN
 F 1 "USB_B_Micro" H 1857 2976 50  0000 C CNN
-F 2 "Connector_USB:USB_Micro-B_Molex-105017-0001" H 1950 2550 50  0001 C CNN
+F 2 "Connector_USB:USB_Micro-B_Molex_47346-0001" H 1950 2550 50  0001 C CNN
 F 3 "~" H 1950 2550 50  0001 C CNN
 	1    1800 2600
